File: KiCad/Kaboom_box_bottom.kicad_pcb (KiCad board)
At the start: 2 copper layers, 150 x 140 mm, 124 parts, among them J101 2mm_clamp, J102 2mm_clamp, J103 2mm_clamp, J104 2mm_clamp, J105 2mm_clamp, J106 2mm_clamp, J107 2mm_clamp, J108 2mm_clamp, J109 2mm_clamp, J110 2mm_clamp, J111 2mm_clamp, J112 2mm_clamp, J113 2mm_clamp, J114 2mm_clamp, J115 2mm_clamp, J116 2mm_clamp, J117 2mm_clamp, J118 2mm_clamp, J119 2mm_clamp, J120 2mm_clamp, J121 2mm_clamp, J122 2mm_clamp, J123 2mm_clamp, J124 2mm_clamp, J125 2mm_clamp, J126 2mm_clamp, J127 2mm_clamp, J128 2mm_clamp, J129 2mm_clamp, J162 Screw_Terminal_01x02, P102 HDR-IDC-2_54-2X5P, P104 HDR-IDC-2_54-2X5P, P106 HDR-IDC-2_54-2X5P, U101 SS54_C22452, U102 EC12E1220813, U103 RaspberryPi_Pico, U104 TS-1187A-B-A-B, U105 TS-1187A-B-A-B, U106 AO3400A, U107 WS2812E-MINI-X1, U108 WS2812E-MINI-X1, U109 WS2812E-MINI-X1, U110 WS2812E-MINI-X1, U111 WS2812E-MINI-X1, U112 WS2812E-MINI-X1, U113 WS2812E-MINI-X1, U114 WS2812E-MINI-X1, U115 WS2812E-MINI-X1, U116 WS2812E-MINI-X1, U117 WS2812E-MINI-X1, U118 WS2812E-MINI-X1, U119 WS2812E-MINI-X1, U120 WS2812E-MINI-X1, U121 WS2812E-MINI-X1, U122 WS2812E-MINI-X1, U123 WS2812E-MINI-X1, U124 WS2812E-MINI-X1, U125 WS2812E-MINI-X1, U126 WS2812E-MINI-X1, U127 WS2812E-MINI-X1, U128 WS2812E-MINI-X1, U129 WS2812E-MINI-X1, U130 WS2812E-MINI-X1, U131 WS2812E-MINI-X1, U132 WS2812E-MINI-X1, U133 WS2812E-MINI-X1, U134 WS2812E-MINI-X1, U135 WS2812E-MINI-X1, U136 74HC595D,118, U137 74HC595D,118, U138 74HC595D,118, U139 74HC595D,118, U140 MT-0-103-F001-T000-RS+PJ, U141 MT-0-103-F001-T000-RS+PJ, U142 MT-0-103-F001-T000-RS+PJ, U149 AO3400A

Commit message: Updates for V2
Parts:
- removed D101: 1N5819WS, footprint:SOD-323_L1.8-W1.3-LS2.5-RD
- added C129: CC0603KRX7R9BB104, footprint:C0603, F.Cu at (195.6, 30.4)
- added R150: 0805W8F0000T5E, footprint:R0805, F.Cu at (178.0, 32.0)
- added R151: 1206W4F1000T5E, footprint:R1206, F.Cu at (166.0, 31.0)
- added R152: 1206W4F1000T5E, footprint:R1206, F.Cu at (166.0, 28.0)
- added R153: 0805W8F0000T5E, footprint:R0805, F.Cu at (208.8, 31.6)
- added R154: 0805W8F0000T5E, footprint:R0805, F.Cu at (211.3, 31.6)
- added R155: 0805W8F2000T5E, footprint:R0805, F.Cu at (146.3, 89.6)
- added R156: 1206W4F1000T5E, footprint:R1206, F.Cu at (166.0, 25.0)
- added R157: 1206W4F1000T5E, footprint:R1206, F.Cu at (160.0, 31.0)
- added R158: 1206W4F1000T5E, footprint:R1206, F.Cu at (160.0, 25.0)
- added R159: 1206W4F1000T5E, footprint:R1206, F.Cu at (160.0, 28.0)
- added U179: 74HC14D,653, footprint:SOIC-14_L8.7-W3.9-P1.27-LS6.0-BL, F.Cu at (201.2, 30.5)
- added U180: AO3400A, footprint:SOT-23-3_L2.9-W1.6-P1.90-LS2.8-BR, F.Cu at (175.0, 28.0)
- C113, C114, C115: value 0603B152K500NT -> CL10B102KB8NNNC
- moved R103 49.0 mm to (141.9, 140.7), turned to 90 degrees
- moved R102 46.7 mm to (144.2, 140.7), turned to 90 degrees
- moved c108 41.2 mm to (147.1, 147.6)
- moved H104 20.2 mm to (147.5, 130.0)
- moved U105 12.1 mm to (149.6, 119.0)
- moved U101 4.68 mm to (150.3, 138.6), turned to 180 degrees
- moved U104 4.65 mm to (143.2, 119.0)
- moved R113 3.46 mm to (152.0, 113.2)
- moved U106 3.00 mm to (152.6, 104.4)
- moved D102 2.77 mm to (219.5, 134.1)
- moved BUZ101 2.50 mm to (145.2, 97.8)
- moved C101 2.50 mm to (205.8, 62.5)
- moved C102 2.50 mm to (205.8, 118.2)
- moved C103 2.50 mm to (198.8, 62.5)
- moved C104 2.50 mm to (198.8, 118.2)
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Connections:
- net Board_0-Net-(D101-A) renamed Board_0-Net-(U106-D)
- U103 pad 17: Board_0-/Bottom/RUMBLE -> Board_0-/Bottom/POWER_DRAIN
- U103 pad 19: Board_0-unconnected-(U103-GPIO14-Pad19) -> Board_0-/Bottom/RUMBLE
- U107 pad 1: Board_0-/Bottom/LED_DATA_IN -> Board_0-/Bottom/LEDs Sheet/LED_DATA_IN
Routing:
- net Board_0-/Bottom/POWER_DRAIN: track 0.00 -> 73.3 mm
- net Board_0-Net-(U179-1Y): track 0.00 -> 12.8 mm
- net Board_0-Net-(U106-D): track 8.22 -> 20.7 mm
- net Board_0-Net-(U180-D): track 0.00 -> 12.3 mm
- net Board_0-Net-(U179-2Y): track 0.00 -> 9.61 mm
- net Board_0-/Bottom/LEDs Sheet/LED_DATA_IN: track 0.00 -> 9.42 mm
- net Board_0-GND: track 50.5 -> 41.1 mm, vias 187 -> 135
- net Board_0-/Bottom/+3.3V: track 416.4 -> 408.4 mm
- net Board_0-/I2C1_SDA_BOT: track 263.9 -> 269.5 mm
- net Board_0-/Bottom/RUMBLE: track 91.5 -> 86.2 mm
- net Board_0-Net-(U106-G): track 2.54 -> 7.75 mm
- net Board_0-/I2C_SCL_BOT: track 260.5 -> 265.7 mm
- net Board_0-/Bottom/BUZZER: track 9.73 -> 4.71 mm
- net Board_0-Net-(U103-3V3_EN): track 10.9 -> 15.3 mm
- net Board_0-Net-(U103-RUN): track 10.6 -> 14.8 mm
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- added copper zone on F.Cu, net Board_0-Net-(R151-Pad2)
Other:
- board size 150 x 140 mm -> 145 x 140 mm
