File: KiCad/Top.kicad_sch (KiCad schematic)
At the start: 2 parts

Commit message: Ready for review
Parts:
- added H? (x4): MountingHole, MountingHole:MountingHole_4.3mm_M4, symbol Mechanical:MountingHole
Connections:
- net +3.3V renamed +3.3V_OLED
Changed lines of the file:
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@@
     (stroke (width 0) (type default))
   )
-  (hierarchical_label "+3.3V" (shape input) (at 96.52 99.06 0) (fields_autoplaced)
+  (hierarchical_label "+3.3V_SHIFT" (shape input) (at 96.52 99.06 0) (fields_autoplaced)
     (effects (font (size 1.27 1.27)) (justify left))
   )
@@
     (effects (font (size 1.27 1.27)) (justify right))
   )
-  (hierarchical_label "+3.3V" (shape input) (at 124.46 88.9 180) (fields_autoplaced)
+  (hierarchical_label "+3.3V_OLED" (shape input) (at 124.46 88.9 180) (fields_autoplaced)
     (effects (font (size 1.27 1.27)) (justify right))
   )
@@
     (effects (font (size 1.27 1.27)) (justify left))
   )
+  (symbol (lib_id "Mechanical:MountingHole") (at 204.47 137.16 0) (unit 1)
+    (in_bom yes) (on_board yes) (dnp no) (fields_autoplaced)
+    (property "Reference" "H?" (at 207.01 135.89 0)
+      (effects (font (size 1.27 1.27)) (justify left))
+    )
+    (property "Value" "MountingHole" (at 207.01 138.43 0)
+      (effects (font (size 1.27 1.27)) (justify left))
+    )
+    (property "Footprint" "MountingHole:MountingHole_4.3mm_M4" (at 204.47 137.16 0)
+      (effects (font (size 1.27 1.27)) hide)
+    )
+    (property "Datasheet" "~" (at 204.47 137.16 0)
+      (effects (font (size 1.27 1.27)) hide)
+    )
+    (instances
+      (project "Kaboom_box"
+        (path "/8d340784-229e-46d1-990c-7f8852f9fc49"
+          (reference "H?") (unit 1)
+        )
+        (path "/8d340784-229e-46d1-990c-7f8852f9fc49/d111de2c-3c3c-486e-8c4b-bd3963817676"
+          (reference "H104") (unit 1)
+        )
+        (path "/8d340784-229e-46d1-990c-7f8852f9fc49/c9ccc42e-41d9-40f0-918f-9c4b4cc23369"
+          (reference "H108") (unit 1)
+        )
+      )
+    )
+  )
+  (symbol (lib_id "Mechanical:MountingHole") (at 204.47 130.81 0) (unit 1)
+    (in_bom yes) (on_board yes) (dnp no) (fields_autoplaced)
+    (property "Reference" "H?" (at 207.01 129.54 0)
+      (effects (font (size 1.27 1.27)) (justify left))
+    )
+    (property "Value" "MountingHole" (at 207.01 132.08 0)
+      (effects (font (size 1.27 1.27)) (justify left))
+    )
+    (property "Footprint" "MountingHole:MountingHole_4.3mm_M4" (at 204.47 130.81 0)
+      (effects (font (size 1.27 1.27)) hide)
+    )
+    (property "Datasheet" "~" (at 204.47 130.81 0)
+      (effects (font (size 1.27 1.27)) hide)
+    )
+    (instances
+      (project "Kaboom_box"
+        (path "/8d340784-229e-46d1-990c-7f8852f9fc49"
+          (reference "H?") (unit 1)
+        )
+        (path "/8d340784-229e-46d1-990c-7f8852f9fc49/d111de2c-3c3c-486e-8c4b-bd3963817676"
+          (reference "H102") (unit 1)
+        )
+        (path "/8d340784-229e-46d1-990c-7f8852f9fc49/c9ccc42e-41d9-40f0-918f-9c4b4cc23369"
+          (reference "H107") (unit 1)
+        )
+      )
+    )
+  )
+  (symbol (lib_id "Mechanical:MountingHole") (at 184.15 137.16 0) (unit 1)
+    (in_bom yes) (on_board yes) (dnp no) (fields_autoplaced)
+    (property "Reference" "H?" (at 186.69 135.89 0)
+      (effects (font (size 1.27 1.27)) (justify left))
+    )
+    (property "Value" "MountingHole" (at 186.69 138.43 0)
+      (effects (font (size 1.27 1.27)) (justify left))
+    )
+    (property "Footprint" "MountingHole:MountingHole_4.3mm_M4" (at 184.15 137.16 0)
+      (effects (font (size 1.27 1.27)) hide)
+    )
+    (property "Datasheet" "~" (at 184.15 137.16 0)
+      (effects (font (size 1.27 1.27)) hide)
+    )
+    (instances
+      (project "Kaboom_box"
+        (path "/8d340784-229e-46d1-990c-7f8852f9fc49"
+          (reference "H?") (unit 1)
+        )
+        (path "/8d340784-229e-46d1-990c-7f8852f9fc49/d111de2c-3c3c-486e-8c4b-bd3963817676"
+          (reference "H103") (unit 1)
+        )
+        (path "/8d340784-229e-46d1-990c-7f8852f9fc49/c9ccc42e-41d9-40f0-918f-9c4b4cc23369"
+          (reference "H106") (unit 1)
+        )
+      )
+    )
+  )
+  (symbol (lib_id "Mechanical:MountingHole") (at 184.15 130.81 0) (unit 1)
+    (in_bom yes) (on_board yes) (dnp no) (fields_autoplaced)
+    (property "Reference" "H?" (at 186.69 129.54 0)
+      (effects (font (size 1.27 1.27)) (justify left))
+    )
+    (property "Value" "MountingHole" (at 186.69 132.08 0)
+      (effects (font (size 1.27 1.27)) (justify left))
+    )
+    (property "Footprint" "MountingHole:MountingHole_4.3mm_M4" (at 184.15 130.81 0)
+      (effects (font (size 1.27 1.27)) hide)
+    )
+    (property "Datasheet" "~" (at 184.15 130.81 0)
+      (effects (font (size 1.27 1.27)) hide)
+    )
+    (instances
+      (project "Kaboom_box"
+        (path "/8d340784-229e-46d1-990c-7f8852f9fc49"
+          (reference "H?") (unit 1)
+        )
+        (path "/8d340784-229e-46d1-990c-7f8852f9fc49/d111de2c-3c3c-486e-8c4b-bd3963817676"
+          (reference "H101") (unit 1)
+        )
+        (path "/8d340784-229e-46d1-990c-7f8852f9fc49/c9ccc42e-41d9-40f0-918f-9c4b4cc23369"
+          (reference "H105") (unit 1)
+        )
+      )
+    )
+  )
   (symbol (lib_id "PZ254V-11-04P_C2691448:PZ254V-11-04P_C2691448") (at 133.35 101.6 0) (unit 1)

Commit message: Updated to generate JLCPCB files
Parts:
- added C127: RVT0J102M0810, footprint:CAP-SMD_BD8.0-L8.3-W8.3-FD, symbol RVT0J102M0810:RVT0J102M0810
Connections:
- net GND: now also C127.2
- net VDD: now also C127.1
Changed lines of the file:
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@@
+    (effects (font (size 1.27 1.27)) (justify right))
+  )
+  (hierarchical_label "GND" (shape input) (at 118.11 137.16 270) (fields_autoplaced)
     (effects (font (size 1.27 1.27)) (justify right))
   )
@@
   )
   (hierarchical_label "GND" (shape input) (at 96.52 135.89 0) (fields_autoplaced)
+    (effects (font (size 1.27 1.27)) (justify left))
+  )
+  (hierarchical_label "VDD" (shape input) (at 118.11 129.54 90) (fields_autoplaced)
     (effects (font (size 1.27 1.27)) (justify left))
   )
@@
         )
       )
+    )
+  )
+  (symbol (lib_id "RVT0J102M0810:RVT0J102M0810") (at 118.11 133.35 0) (unit 1)
+    (in_bom yes) (on_board yes) (dnp no) (fields_autoplaced)
+    (property "Reference" "C127" (at 121.92 130.8139 0)
+      (effects (font (size 1.27 1.27)) (justify left))
+    )
+    (property "Value" "RVT0J102M0810" (at 121.92 133.3539 0)
+      (effects (font (size 1.27 1.27)) (justify left))
+    )
+    (property "Footprint" "footprint:CAP-SMD_BD8.0-L8.3-W8.3-FD" (at 118.11 143.51 0)
+      (effects (font (size 1.27 1.27) italic) hide)
+    )
+    (property "Datasheet" "https://item.szlcsc.com/245644.html" (at 115.824 133.223 0)
+      (effects (font (size 1.27 1.27)) (justify left) hide)
+    )
+    (property "LCSC" "C42851" (at 118.11 133.35 0)
+      (effects (font (size 1.27 1.27)) hide)
+    )
+    (pin "1")
+    (pin "2")
+    (instances
+      (project "Kaboom_box"
+        (path "/8d340784-229e-46d1-990c-7f8852f9fc49/d111de2c-3c3c-486e-8c4b-bd3963817676"
+          (reference "C127") (unit 1)
+        )
+        (path "/8d340784-229e-46d1-990c-7f8852f9fc49/c9ccc42e-41d9-40f0-918f-9c4b4cc23369"
+          (reference "C128") (unit 1)
+        )
+      )

Commit message: Updates for V2
Connections:
- net +3.3V_OLED: now also U?.2
- net GND: now also U?.1
- net I2C1_SCL: now also U?.3
- net I2C1_SDA: now also U?.4
Other:
- moved on the sheet: U?
Changed lines of the file:
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@@
-    (stroke (width 0) (type default))
-  )
-  (wire (pts (xy 124.46 88.9) (xy 127 88.9))
     (stroke (width 0) (type default))
   )
@@
     (stroke (width 0) (type default))
   )
+  (wire (pts (xy 143.51 90.17) (xy 163.83 90.17))
+    (stroke (width 0) (type default))
+  )
   (wire (pts (xy 93.98 86.36) (xy 96.52 86.36))
     (stroke (width 0) (type default))
   )
-  (wire (pts (xy 124.46 91.44) (xy 127 91.44))
-    (stroke (width 0) (type default))
-  )
-  (wire (pts (xy 124.46 86.36) (xy 127 86.36))
-    (stroke (width 0) (type default))
-  )
-  (wire (pts (xy 124.46 83.82) (xy 127 83.82))
+  (wire (pts (xy 143.51 85.09) (xy 163.83 85.09))
+    (stroke (width 0) (type default))
+  )
+  (wire (pts (xy 143.51 87.63) (xy 163.83 87.63))
+    (stroke (width 0) (type default))
+  )
+  (wire (pts (xy 143.51 82.55) (xy 163.83 82.55))
     (stroke (width 0) (type default))
   )
@@
     (effects (font (size 1.27 1.27)) (justify left))
   )
-  (hierarchical_label "I2C1_SDA" (shape input) (at 124.46 83.82 180) (fields_autoplaced)
-    (effects (font (size 1.27 1.27)) (justify right))
-  )
-  (hierarchical_label "GND" (shape input) (at 124.46 91.44 180) (fields_autoplaced)
-    (effects (font (size 1.27 1.27)) (justify right))
-  )
-  (hierarchical_label "+3.3V_OLED" (shape input) (at 124.46 88.9 180) (fields_autoplaced)
+  (hierarchical_label "I2C1_SDA" (shape input) (at 161.29 82.55 180) (fields_autoplaced)
+    (effects (font (size 1.27 1.27)) (justify right))
+  )
+  (hierarchical_label "GND" (shape input) (at 161.29 90.17 180) (fields_autoplaced)
+    (effects (font (size 1.27 1.27)) (justify right))
+  )
+  (hierarchical_label "+3.3V_OLED" (shape input) (at 161.29 87.63 180) (fields_autoplaced)
     (effects (font (size 1.27 1.27)) (justify right))
   )
@@
     (effects (font (size 1.27 1.27)) (justify right))
   )
-  (hierarchical_label "I2C1_SCL" (shape input) (at 124.46 86.36 180) (fields_autoplaced)
+  (hierarchical_label "I2C1_SCL" (shape input) (at 161.29 85.09 180) (fields_autoplaced)
     (effects (font (size 1.27 1.27)) (justify right))
   )
@@
     )
   )
-  (symbol (lib_id "PZ254V-11-04P_C2691448:PZ254V-11-04P_C2691448") (at 133.35 101.6 0) (unit 1)
-    (in_bom yes) (on_board no) (dnp no) (fields_autoplaced)
-    (property "Reference" "U?" (at 137.16 100.33 0)
-      (effects (font (size 1.27 1.27)) (justify left))
-    )
-    (property "Value" "PZ254V-11-04P_C2691448" (at 137.16 102.87 0)
-      (effects (font (size 1.27 1.27)) (justify left))
-    )
-    (property "Footprint" "footprint:HDR-TH_4P-P2.54-V-M" (at 133.35 111.76 0)
+  (symbol (lib_id "PZ254V-11-04P_C2691448:PZ254V-11-04P_C2691448") (at 138.43 86.36 180) (unit 1)
+    (in_bom yes) (on_board yes) (dnp no) (fields_autoplaced)
+    (property "Reference" "U?" (at 138.43 74.93 0)
+      (effects (font (size 1.27 1.27)))
+    )
+    (property "Value" "PZ254V-11-04P_C2691448" (at 138.43 77.47 0)
+      (effects (font (size 1.27 1.27)))
+    )
+    (property "Footprint" "footprint:HDR-TH_4P-P2.54-V-M" (at 138.43 76.2 0)
       (effects (font (size 1.27 1.27) italic) hide)
     )
-    (property "Datasheet" "https://item.szlcsc.com/502959.html" (at 131.064 101.473 0)
+    (property "Datasheet" "https://item.szlcsc.com/502959.html" (at 140.716 86.487 0)
       (effects (font (size 1.27 1.27)) (justify left) hide)
     )
-    (property "LCSC" "C2691448" (at 133.35 101.6 0)
+    (property "LCSC" "C2691448" (at 138.43 86.36 0)
       (effects (font (size 1.27 1.27)) hide)
     )
@@
     )
   )
-  (symbol (lib_id "HS96L03W2C03:HS96L03W2C03") (at 133.35 87.63 0) (mirror x) (unit 1)
+  (symbol (lib_id "HS96L03W2C03:HS96L03W2C03") (at 170.18 86.36 0) (mirror x) (unit 1)
     (in_bom yes) (on_board yes) (dnp no)
-    (property "Reference" "U?" (at 138.43 88.9 0)
-      (effects (font (size 1.27 1.27)) (justify left))
-    )
-    (property "Value" "HS96L03W2C03" (at 138.43 86.36 0)
-      (effects (font (size 1.27 1.27)) (justify left))
-    )
-    (property "Footprint" "footprint:OLED-TH_L27.8-W27.2-P2.54_C9900033791" (at 133.35 77.47 0)
+    (property "Reference" "U?" (at 175.26 87.63 0)
+      (effects (font (size 1.27 1.27)) (justify left))
+    )
+    (property "Value" "HS96L03W2C03" (at 175.26 85.09 0)
+      (effects (font (size 1.27 1.27)) (justify left))
+    )
+    (property "Footprint" "footprint:OLED-TH_L27.8-W27.2-P2.54_C9900033791" (at 170.18 76.2 0)
       (effects (font (size 1.27 1.27) italic) hide)
     )
-    (property "Datasheet" "https://img.jlc.com/image//data/smt-stock-produce/componentSizePhoto/2022-11-01/43d81eb4655044fe9599202a8cead0a7/BG2211010127_D22103102259_back.png" (at 131.064 87.757 0)
+    (property "Datasheet" "https://img.jlc.com/image//data/smt-stock-produce/componentSizePhoto/2022-11-01/43d81eb4655044fe9599202a8cead0a7/BG2211010127_D22103102259_back.png" (at 167.894 86.487 0)
       (effects (font (size 1.27 1.27)) (justify left) hide)
     )
-    (property "LCSC" "C5248080" (at 133.35 87.63 0)
-      (effects (font (size 1.27 1.27)) hide)
-    )
+    (property "LCSC" "C5248080" (at 170.18 86.36 0)
+      (effects (font (size 1.27 1.27)) hide)
+    )

Commit message: First production
Parts:
- gave numbers to parts that had none: 6
- renumbered C127 to C128
