File: KiCad/Kaboom_box.kicad_pcb (KiCad board)
At the start: 2 copper layers, 351.5 x 141.5 mm, 207 parts, among them J101 2mm_clamp, J102 2mm_clamp, J103 2mm_clamp, J104 2mm_clamp, J105 2mm_clamp, J106 2mm_clamp, J107 2mm_clamp, J108 2mm_clamp, J109 2mm_clamp, J110 2mm_clamp, J111 2mm_clamp, J112 2mm_clamp, J113 2mm_clamp, J114 2mm_clamp, J115 2mm_clamp, J116 2mm_clamp, J117 2mm_clamp, J118 2mm_clamp, J119 2mm_clamp, J120 2mm_clamp, J121 2mm_clamp, J122 2mm_clamp, J123 2mm_clamp, J124 2mm_clamp, J125 2mm_clamp, J126 2mm_clamp, J127 2mm_clamp, J128 2mm_clamp, J129 2mm_clamp, J130 2mm_clamp, J131 2mm_clamp, J132 2mm_clamp, J133 2mm_clamp, J134 2mm_clamp, J135 2mm_clamp, J136 2mm_clamp, J137 2mm_clamp, J138 2mm_clamp, J139 2mm_clamp, J140 2mm_clamp, J141 2mm_clamp, J142 2mm_clamp, J143 2mm_clamp, J144 2mm_clamp, J145 2mm_clamp, J146 2mm_clamp, J147 2mm_clamp, J148 2mm_clamp, J149 2mm_clamp, J150 2mm_clamp, J151 2mm_clamp, J152 2mm_clamp, J153 2mm_clamp, J154 2mm_clamp, J155 2mm_clamp, J156 2mm_clamp, J157 2mm_clamp, J158 2mm_clamp, J162 Screw_Terminal_01x02, P101 HDR-IDC-2_54-2X5P, P102 HDR-IDC-2_54-2X5P, P103 HDR-IDC-2_54-2X5P, P104 HDR-IDC-2_54-2X5P, P105 HDR-IDC-2_54-2X5P, P106 HDR-IDC-2_54-2X5P, U101 SS54_C22452, U102 EC12E1220813, U103 RaspberryPi_Pico, U104 TS-1187A-B-A-B, U105 TS-1187A-B-A-B, U106 AO3400A, U107 WS2812E-MINI-X1, U108 WS2812E-MINI-X1, U109 WS2812E-MINI-X1, U110 WS2812E-MINI-X1, U111 WS2812E-MINI-X1, U112 WS2812E-MINI-X1, U113 WS2812E-MINI-X1, U114 WS2812E-MINI-X1, U115 WS2812E-MINI-X1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

Commit message: UPdated outline + added pull down resistors on input of shifts
Parts:
- removed D101: 1N5819WS, footprint:SOD-323_L1.8-W1.3-LS2.5-RD
- added R121: 0603WAF1202T5E, footprint:R0603, F.Cu at (312.0, 82.0)
- added R122: 0603WAF1202T5E, footprint:R0603, F.Cu at (312.0, 96.0)
- added R123: 0603WAF1202T5E, footprint:R0603, F.Cu at (312.0, 110.0)
- added R124: 0603WAF1202T5E, footprint:R0603, F.Cu at (312.0, 124.0)
- added R125: 0603WAF1202T5E, footprint:R0603, F.Cu at (312.0, 138.0)
- added R126: 0603WAF1202T5E, footprint:R0603, F.Cu at (312.0, 152.0)
- added R127: 0603WAF1202T5E, footprint:R0603, F.Cu at (312.0, 166.0)
- added R128: 0603WAF1202T5E, footprint:R0603, F.Cu at (312.0, 180.0)
- added R129: 0603WAF1202T5E, footprint:R0603, F.Cu at (312.0, 80.0)
- added R130: 0603WAF1202T5E, footprint:R0603, F.Cu at (312.0, 94.0)
- added R131: 0603WAF1202T5E, footprint:R0603, F.Cu at (312.0, 108.0)
- added R132: 0603WAF1202T5E, footprint:R0603, F.Cu at (312.0, 122.0)
- added R133: 0603WAF1202T5E, footprint:R0603, F.Cu at (312.0, 136.0)
- added R134: 0603WAF1202T5E, footprint:R0603, F.Cu at (312.0, 150.0)
- added R135: 0603WAF1202T5E, footprint:R0603, F.Cu at (312.0, 164.0)
- added R136: 0603WAF1202T5E, footprint:R0603, F.Cu at (312.0, 178.0)
- added R137: 0603WAF1202T5E, footprint:R0603, F.Cu at (279.0, 82.0)
- added R138: 0603WAF1202T5E, footprint:R0603, F.Cu at (279.0, 96.0)
- added R139: 0603WAF1202T5E, footprint:R0603, F.Cu at (279.0, 110.0)
- added R140: 0603WAF1202T5E, footprint:R0603, F.Cu at (279.0, 124.0)
- added R141: 0603WAF1202T5E, footprint:R0603, F.Cu at (279.0, 138.0)
- added R142: 0603WAF1202T5E, footprint:R0603, F.Cu at (279.0, 152.0)
- added R143: 0603WAF1202T5E, footprint:R0603, F.Cu at (279.0, 166.0)
- added R144: 0603WAF1202T5E, footprint:R0603, F.Cu at (279.0, 180.0)
- added R145: 0603WAF1202T5E, footprint:R0603, F.Cu at (279.0, 80.0)
- added R146: 0603WAF1202T5E, footprint:R0603, F.Cu at (279.0, 94.0)
- added R147: 0603WAF1202T5E, footprint:R0603, F.Cu at (279.0, 108.0)
- added R148: 0603WAF1202T5E, footprint:R0603, F.Cu at (279.0, 122.0)
- added R149: 0603WAF1202T5E, footprint:R0603, F.Cu at (279.0, 136.0)
- added R150: 0805W8F0000T5E, footprint:R0805, F.Cu at (95.5, 72.0)
- added R151: 1206W4F1000T5E, footprint:R1206, F.Cu at (83.5, 71.0)
- added R152: 1206W4F1000T5E, footprint:R1206, F.Cu at (83.5, 68.0)
- added R153: 0805W8F0000T5E, footprint:R0805, F.Cu at (125.3, 71.7)
- added R154: 0805W8F0000T5E, footprint:R0805, F.Cu at (127.8, 71.7)
- added R155: 0805W8F2000T5E, footprint:R0805, F.Cu at (63.8, 129.6)
- added R156: 1206W4F1000T5E, footprint:R1206, F.Cu at (83.5, 65.0)
- added R157: 1206W4F1000T5E, footprint:R1206, F.Cu at (77.5, 71.0)
- added R158: 1206W4F1000T5E, footprint:R1206, F.Cu at (77.5, 65.0)
- added R159: 1206W4F1000T5E, footprint:R1206, F.Cu at (77.5, 68.0)
- added U179: 74HC14D,653, footprint:SOIC-14_L8.7-W3.9-P1.27-LS6.0-BL, F.Cu at (118.7, 70.5)
- added U180: AO3400A, footprint:SOT-23-3_L2.9-W1.6-P1.90-LS2.8-BR, F.Cu at (92.5, 68.0)
- moved R103 46.5 mm to (59.4, 180.7), turned to 90 degrees
- moved R102 44.2 mm to (61.7, 180.7), turned to 90 degrees
- moved c108 38.7 mm to (64.6, 187.6)
- moved H104 20.6 mm to (65.0, 170.0)
- moved U105 12.6 mm to (67.1, 159.0)
- moved H105 10.0 mm to (381.5, 71.5)
- moved H107 10.0 mm to (381.5, 191.5)
- moved U106 5.05 mm to (70.0, 144.4)
- moved H102 5.00 mm to (65.0, 70.0)
- moved KEY101 5.00 mm to (71.6, 88.4)
- moved R106 5.00 mm to (62.4, 106.0)
- moved R107 5.00 mm to (62.3, 122.0)
- moved R112 5.00 mm to (71.1, 98.3)
- moved U102 5.00 mm to (63.8, 114.0)
- moved U144 5.00 mm to (384.2, 130.0)
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Connections:
- U103 pad 17: /Bottom/RUMBLE -> /Bottom/POWER_DRAIN
- U103 pad 19: unconnected-(U103-GPIO14-Pad19) -> /Bottom/RUMBLE
- U107 pad 1: /Bottom/LED_DATA_IN -> /Bottom/LEDs Sheet/LED_DATA_IN
Routing:
- net /Bottom/POWER_DRAIN: track 0.00 -> 73.3 mm
- net Net-(U106-D): track 8.22 -> 20.7 mm
- net Net-(U180-D): track 0.00 -> 12.3 mm
- net Net-(U179-1Y): track 0.00 -> 11.8 mm
- net /Bottom/LEDs Sheet/LED_DATA_IN: track 0.00 -> 9.79 mm
- net GND: track 50.5 -> 41.1 mm, vias 187 -> 122
- net /Bottom/VDD: track 1162.8 -> 1153.8 mm
- net Net-(U179-2Y): track 0.00 -> 8.85 mm
- net /Bottom/+3.3V: track 416.4 -> 408.4 mm
- net /Top/Shift_Parallel_to_Serial/J157: track 23.8 -> 30.4 mm
- net /Top/Shift_Parallel_to_Serial/J158: track 23.7 -> 30.4 mm
- net /Top/Shift_Parallel_to_Serial/J156: track 23.6 -> 30.3 mm
- net /Top/Shift_Parallel_to_Serial/J155: track 23.8 -> 30.5 mm
- net /Top/Shift_Parallel_to_Serial/J154: track 23.9 -> 30.6 mm
- net /Top/Shift_Parallel_to_Serial/J153: track 9.28 -> 15.9 mm
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- added copper zone on F.Cu, net Net-(R151-Pad2)
Other:
- board size 351.5 x 141.5 mm -> 336.5 x 141.5 mm

Commit message: Updates for V2
Parts:
- added C129: CC0603KRX7R9BB104, footprint:C0603, F.Cu at (113.0, 70.5)
- added U143: PZ254V-11-04P_C2691448, footprint:HDR-TH_4P-P2.54-V-M, F.Cu at (384.2, 130.0)
- C113, C114, C115: value 0603B152K500NT -> CL10B102KB8NNNC
- moved C128 1.97 mm to (363.3, 71.2)
- moved R154 1.03 mm to (128.8, 71.7)
- moved R153 1.03 mm to (126.3, 71.7)
- moved D102 0.63 mm to (137.0, 174.1)
Routing:
- net /Bottom/VDD: track 1153.8 -> 1163.8 mm
- net /Top/LED_DATA_IN: track 130.0 -> 131.9 mm
- net /Top/VDD: track 587.4 -> 588.5 mm
- net /Top/+3.3V_OLED: track 252.6 -> 251.6 mm
- net Net-(U179-1Y): track 11.8 -> 12.8 mm
- net Net-(U179-2Y): track 8.85 -> 9.61 mm
- net GND: vias 122 -> 135
- net /Top/GND: vias 135 -> 232
Other:
- board size 336.5 x 141.5 mm -> 333.9 x 141.1 mm

Commit message: Ready for PCB layout with discreet LEDs
Parts:
- removed C101: CC0603KRX7R9BB104, footprint:C0603
- removed the C102 at (123.2, 158.2)
- removed the C104 at (116.2, 158.2)
- removed the C105 at (109.0, 102.5)
- removed the C106 at (109.0, 158.0)
- removed the C107 at (101.5, 102.5)
- removed D102: 1N5819WS, footprint:SOD-323_L1.8-W1.3-LS2.5-RD
- removed J162: Screw_Terminal_01x02, TerminalBlock_Phoenix:TerminalBlock_Phoenix_MKDS-1,5-2_1x02_P5.00mm_Horizontal
- removed the R113 at (69.5, 153.2)
- removed the R120 at (134.8, 181.7)
- removed the R153 at (126.3, 71.7)
- removed the R154 at (128.8, 71.7)
- removed the U106 at (70.0, 144.4)
- removed the U108 at (126.0, 95.0)
- removed the U109 at (126.0, 109.0)
- removed the U110 at (126.0, 123.0)
- removed the U111 at (126.0, 137.0)
- removed the U112 at (126.0, 151.0)
- removed the U113 at (126.0, 165.0)
- removed the U114 at (126.0, 179.0)
- removed the U115 at (119.0, 81.0)
- removed the U116 at (119.0, 95.0)
- removed the U117 at (119.0, 109.0)
- removed the U118 at (119.0, 123.0)
- removed the U119 at (119.0, 137.0)
- removed the U120 at (119.0, 151.0)
- added C116: CC0603KRX7R9BB104, footprint:C0603, F.Cu at (237.7, -34.9)
- added C117: CC0603KRX7R9BB104, footprint:C0603, F.Cu at (237.7, -48.2)
- added C118: CC0603KRX7R9BB104, footprint:C0603, F.Cu at (251.3, -34.9)
- added C119: CC0603KRX7R9BB104, footprint:C0603, F.Cu at (237.7, -61.5)
- added C127: CC0603KRX7R9BB104, footprint:C0603, F.Cu at (430.8, -50.5)
- added C128: CC0603KRX7R9BB104, footprint:C0603, F.Cu at (430.8, -37.2)
- added C130: CC0603KRX7R9BB104, footprint:C0603, F.Cu at (430.8, -23.9)
- added D101: 1N5819WS, footprint:SOD-323_L1.8-W1.3-LS2.5-RD, F.Cu at (33.4, 138.5)
- added J159: Screw_Terminal_01x02, TerminalBlock_Phoenix:TerminalBlock_Phoenix_MKDS-1,5-2_1x02_P5.00mm_Horizontal, F.Cu at (34.8, 131.3)
- added LED104: KT-0603R, footprint:LED0603-RD, F.Cu at (301.2, -28.5)
- added LED105: KT-0603R, footprint:LED0603-RD, F.Cu at (301.2, -25.9)
- added LED106: KT-0603R, footprint:LED0603-RD, F.Cu at (301.2, -23.2)
- added LED107: KT-0603R, footprint:LED0603-RD, F.Cu at (28.3, 130.5)
- added LED108: KT-0603R, footprint:LED0603-RD, F.Cu at (28.3, 133.1)
- added LED109: KT-0603R, footprint:LED0603-RD, F.Cu at (301.2, -38.9)
- added LED110: KT-0603R, footprint:LED0603-RD, F.Cu at (301.2, -36.3)
- added LED111: KT-0603R, footprint:LED0603-RD, F.Cu at (301.2, -33.6)
- added LED112: KT-0603R, footprint:LED0603-RD, F.Cu at (272.7, -90.9)
- added LED113: KT-0603R, footprint:LED0603-RD, F.Cu at (272.7, -88.3)
- added LED114: KT-0603R, footprint:LED0603-RD, F.Cu at (272.7, -85.6)
- added LED115: KT-0603R, footprint:LED0603-RD, F.Cu at (286.9, -90.9)
- added LED116: KT-0603R, footprint:LED0603-RD, F.Cu at (286.9, -88.3)
- added LED117: KT-0603R, footprint:LED0603-RD, F.Cu at (286.9, -85.6)
- added LED118: KT-0603R, footprint:LED0603-RD, F.Cu at (315.4, -90.9)
- added LED119: KT-0603R, footprint:LED0603-RD, F.Cu at (315.4, -88.3)
- added LED120: KT-0603R, footprint:LED0603-RD, F.Cu at (315.4, -85.6)
- added LED121: KT-0603R, footprint:LED0603-RD, F.Cu at (301.2, -90.9)
- added LED122: KT-0603R, footprint:LED0603-RD, F.Cu at (301.2, -88.3)
- added LED123: KT-0603R, footprint:LED0603-RD, F.Cu at (301.2, -85.6)
- added LED124: KT-0603R, footprint:LED0603-RD, F.Cu at (286.9, -70.1)
- added LED125: KT-0603R, footprint:LED0603-RD, F.Cu at (286.9, -67.5)
- added LED126: KT-0603R, footprint:LED0603-RD, F.Cu at (286.9, -64.8)
- added LED127: KT-0603R, footprint:LED0603-RD, F.Cu at (272.7, -38.9)
- added LED128: KT-0603R, footprint:LED0603-RD, F.Cu at (272.7, -36.3)
- added LED129: KT-0603R, footprint:LED0603-RD, F.Cu at (272.7, -33.6)
- added LED130: KT-0603R, footprint:LED0603-RD, F.Cu at (272.7, -28.5)
- added LED131: KT-0603R, footprint:LED0603-RD, F.Cu at (272.7, -25.9)
- added LED132: KT-0603R, footprint:LED0603-RD, F.Cu at (272.7, -23.2)
- added LED133: KT-0603R, footprint:LED0603-RD, F.Cu at (301.2, -59.7)
- added LED134: KT-0603R, footprint:LED0603-RD, F.Cu at (301.2, -57.1)
- added LED135: KT-0603R, footprint:LED0603-RD, F.Cu at (301.2, -54.4)
- added LED136: KT-0603R, footprint:LED0603-RD, F.Cu at (286.9, -59.7)
- added LED137: KT-0603R, footprint:LED0603-RD, F.Cu at (286.9, -57.1)
- added LED138: KT-0603R, footprint:LED0603-RD, F.Cu at (286.9, -54.4)
- added LED139: KT-0603R, footprint:LED0603-RD, F.Cu at (315.4, -28.5)
- added LED140: KT-0603R, footprint:LED0603-RD, F.Cu at (315.4, -25.9)
- added LED141: KT-0603R, footprint:LED0603-RD, F.Cu at (315.4, -23.2)
- added LED142: KT-0603R, footprint:LED0603-RD, F.Cu at (272.7, -101.3)
- added LED143: KT-0603R, footprint:LED0603-RD, F.Cu at (272.7, -98.7)
- added LED144: KT-0603R, footprint:LED0603-RD, F.Cu at (272.7, -96.0)
- added LED145: KT-0603R, footprint:LED0603-RD, F.Cu at (286.9, -101.3)
- added LED146: KT-0603R, footprint:LED0603-RD, F.Cu at (286.9, -98.7)
- added LED147: KT-0603R, footprint:LED0603-RD, F.Cu at (286.9, -96.0)
- added LED148: KT-0603R, footprint:LED0603-RD, F.Cu at (315.4, -101.3)
- added LED149: KT-0603R, footprint:LED0603-RD, F.Cu at (315.4, -98.7)
- added LED150: KT-0603R, footprint:LED0603-RD, F.Cu at (315.4, -96.0)
- added LED151: KT-0603R, footprint:LED0603-RD, F.Cu at (301.2, -101.3)
- added LED152: KT-0603R, footprint:LED0603-RD, F.Cu at (301.2, -98.7)
- added LED153: KT-0603R, footprint:LED0603-RD, F.Cu at (301.2, -96.0)
- added LED154: KT-0603R, footprint:LED0603-RD, F.Cu at (315.4, -70.1)
- added LED155: KT-0603R, footprint:LED0603-RD, F.Cu at (315.4, -67.5)
- added LED156: KT-0603R, footprint:LED0603-RD, F.Cu at (315.4, -64.8)
- added LED157: KT-0603R, footprint:LED0603-RD, F.Cu at (272.7, -49.3)
- added LED158: KT-0603R, footprint:LED0603-RD, F.Cu at (272.7, -46.7)
- added LED159: KT-0603R, footprint:LED0603-RD, F.Cu at (272.7, -44.0)
- added LED160: KT-0603R, footprint:LED0603-RD, F.Cu at (315.4, -59.7)
- added LED161: KT-0603R, footprint:LED0603-RD, F.Cu at (315.4, -57.1)
- added LED162: KT-0603R, footprint:LED0603-RD, F.Cu at (315.4, -54.4)
- added LED163: KT-0603R, footprint:LED0603-RD, F.Cu at (315.4, -38.9)
- added LED164: KT-0603R, footprint:LED0603-RD, F.Cu at (315.4, -36.3)
- added LED165: KT-0603R, footprint:LED0603-RD, F.Cu at (315.4, -33.6)
- added LED166: KT-0603R, footprint:LED0603-RD, F.Cu at (272.7, -59.7)
- added LED167: KT-0603R, footprint:LED0603-RD, F.Cu at (272.7, -57.1)
- added LED168: KT-0603R, footprint:LED0603-RD, F.Cu at (272.7, -54.4)
- added LED169: KT-0603R, footprint:LED0603-RD, F.Cu at (315.4, -49.3)
- added LED170: KT-0603R, footprint:LED0603-RD, F.Cu at (315.4, -46.7)
- added LED171: KT-0603R, footprint:LED0603-RD, F.Cu at (315.4, -44.0)
- added LED172: KT-0603R, footprint:LED0603-RD, F.Cu at (301.2, -70.1)
- added LED173: KT-0603R, footprint:LED0603-RD, F.Cu at (301.2, -67.5)
- added LED174: KT-0603R, footprint:LED0603-RD, F.Cu at (301.2, -64.8)
- added LED175: KT-0603R, footprint:LED0603-RD, F.Cu at (272.7, -80.5)
- added LED176: KT-0603R, footprint:LED0603-RD, F.Cu at (272.7, -77.9)
- added LED177: KT-0603R, footprint:LED0603-RD, F.Cu at (272.7, -75.2)
- added LED178: KT-0603R, footprint:LED0603-RD, F.Cu at (286.9, -80.5)
- added LED179: KT-0603R, footprint:LED0603-RD, F.Cu at (286.9, -77.9)
- added LED180: KT-0603R, footprint:LED0603-RD, F.Cu at (286.9, -75.2)
- added LED181: KT-0603R, footprint:LED0603-RD, F.Cu at (315.4, -80.5)
- added LED182: KT-0603R, footprint:LED0603-RD, F.Cu at (315.4, -77.9)
- added LED183: KT-0603R, footprint:LED0603-RD, F.Cu at (315.4, -75.2)
- added LED184: KT-0603R, footprint:LED0603-RD, F.Cu at (301.2, -80.5)
- added LED185: KT-0603R, footprint:LED0603-RD, F.Cu at (301.2, -77.9)
- added LED186: KT-0603R, footprint:LED0603-RD, F.Cu at (301.2, -75.2)
- added LED187: KT-0603R, footprint:LED0603-RD, F.Cu at (286.9, -49.3)
- added LED188: KT-0603R, footprint:LED0603-RD, F.Cu at (286.9, -46.7)
- added LED189: KT-0603R, footprint:LED0603-RD, F.Cu at (286.9, -44.0)
- added LED190: KT-0603R, footprint:LED0603-RD, F.Cu at (286.9, -38.9)
- added LED191: KT-0603R, footprint:LED0603-RD, F.Cu at (286.9, -36.3)
- added LED192: KT-0603R, footprint:LED0603-RD, F.Cu at (286.9, -33.6)
- added LED193: KT-0603R, footprint:LED0603-RD, F.Cu at (301.2, -49.3)
- added LED194: KT-0603R, footprint:LED0603-RD, F.Cu at (301.2, -46.7)
- added LED195: KT-0603R, footprint:LED0603-RD, F.Cu at (301.2, -44.0)
- added LED196: KT-0603R, footprint:LED0603-RD, F.Cu at (286.9, -28.5)
- added LED197: KT-0603R, footprint:LED0603-RD, F.Cu at (286.9, -25.9)
- added LED198: KT-0603R, footprint:LED0603-RD, F.Cu at (286.9, -23.2)
- added LED199: KT-0603R, footprint:LED0603-RD, F.Cu at (272.7, -70.1)
- added LED200: KT-0603R, footprint:LED0603-RD, F.Cu at (272.7, -67.5)
- added LED201: KT-0603R, footprint:LED0603-RD, F.Cu at (272.7, -64.8)
- added LED202: KT-0603R, footprint:LED0603-RD, F.Cu at (378.8, -79.9)
- added LED203: KT-0603R, footprint:LED0603-RD, F.Cu at (378.8, -77.3)
- added LED204: KT-0603R, footprint:LED0603-RD, F.Cu at (378.8, -74.6)
- added LED205: KT-0603R, footprint:LED0603-RD, F.Cu at (378.8, -69.5)
- added LED206: KT-0603R, footprint:LED0603-RD, F.Cu at (378.8, -66.9)
- added LED207: KT-0603R, footprint:LED0603-RD, F.Cu at (378.8, -64.2)
- added LED208: KT-0603R, footprint:LED0603-RD, F.Cu at (378.8, -48.7)
- added LED209: KT-0603R, footprint:LED0603-RD, F.Cu at (378.8, -46.1)
- added LED210: KT-0603R, footprint:LED0603-RD, F.Cu at (378.8, -43.4)
- added LED211: KT-0603R, footprint:LED0603-RD, F.Cu at (378.8, -59.1)
- added LED212: KT-0603R, footprint:LED0603-RD, F.Cu at (378.8, -56.5)
- added LED213: KT-0603R, footprint:LED0603-RD, F.Cu at (378.8, -53.8)
- added LED214: KT-0603R, footprint:LED0603-RD, F.Cu at (393.0, -27.9)
- added LED215: KT-0603R, footprint:LED0603-RD, F.Cu at (393.0, -25.3)
- added LED216: KT-0603R, footprint:LED0603-RD, F.Cu at (393.0, -22.6)
- added LED217: KT-0603R, footprint:LED0603-RD, F.Cu at (407.3, -79.9)
- added LED218: KT-0603R, footprint:LED0603-RD, F.Cu at (407.3, -77.3)
- added LED219: KT-0603R, footprint:LED0603-RD, F.Cu at (407.3, -74.6)
- added LED220: KT-0603R, footprint:LED0603-RD, F.Cu at (435.7, -79.9)
- added LED221: KT-0603R, footprint:LED0603-RD, F.Cu at (435.7, -77.3)
- added LED222: KT-0603R, footprint:LED0603-RD, F.Cu at (435.7, -74.6)
- added LED223: KT-0603R, footprint:LED0603-RD, F.Cu at (421.5, -79.9)
- added LED224: KT-0603R, footprint:LED0603-RD, F.Cu at (421.5, -77.3)
- added LED225: KT-0603R, footprint:LED0603-RD, F.Cu at (421.5, -74.6)
- added LED226: KT-0603R, footprint:LED0603-RD, F.Cu at (393.0, -79.9)
- added LED227: KT-0603R, footprint:LED0603-RD, F.Cu at (393.0, -77.3)
- added LED228: KT-0603R, footprint:LED0603-RD, F.Cu at (393.0, -74.6)
- added LED229: KT-0603R, footprint:LED0603-RD, F.Cu at (378.8, -90.3)
- added LED230: KT-0603R, footprint:LED0603-RD, F.Cu at (378.8, -87.7)
- added LED231: KT-0603R, footprint:LED0603-RD, F.Cu at (378.8, -85.0)
- added LED232: KT-0603R, footprint:LED0603-RD, F.Cu at (435.7, -90.3)
- added LED233: KT-0603R, footprint:LED0603-RD, F.Cu at (435.7, -87.7)
- added LED234: KT-0603R, footprint:LED0603-RD, F.Cu at (435.7, -85.0)
- added LED235: KT-0603R, footprint:LED0603-RD, F.Cu at (378.8, -38.3)
- added LED236: KT-0603R, footprint:LED0603-RD, F.Cu at (378.8, -35.7)
- added LED237: KT-0603R, footprint:LED0603-RD, F.Cu at (378.8, -33.0)
- added LED238: KT-0603R, footprint:LED0603-RD, F.Cu at (407.3, -48.7)
- added LED239: KT-0603R, footprint:LED0603-RD, F.Cu at (407.3, -46.1)
- added LED240: KT-0603R, footprint:LED0603-RD, F.Cu at (407.3, -43.4)
- added LED241: KT-0603R, footprint:LED0603-RD, F.Cu at (407.3, -38.3)
- added LED242: KT-0603R, footprint:LED0603-RD, F.Cu at (407.3, -35.7)
- added LED243: KT-0603R, footprint:LED0603-RD, F.Cu at (407.3, -33.0)
- added LED244: KT-0603R, footprint:LED0603-RD, F.Cu at (378.8, -100.7)
- added LED245: KT-0603R, footprint:LED0603-RD, F.Cu at (378.8, -98.1)
- added LED246: KT-0603R, footprint:LED0603-RD, F.Cu at (378.8, -95.4)
- added LED247: KT-0603R, footprint:LED0603-RD, F.Cu at (407.3, -27.9)
- added LED248: KT-0603R, footprint:LED0603-RD, F.Cu at (407.3, -25.3)
- added LED249: KT-0603R, footprint:LED0603-RD, F.Cu at (407.3, -22.6)
- added LED250: KT-0603R, footprint:LED0603-RD, F.Cu at (378.8, -27.9)
- added LED251: KT-0603R, footprint:LED0603-RD, F.Cu at (378.8, -25.3)
- added LED252: KT-0603R, footprint:LED0603-RD, F.Cu at (378.8, -22.6)
- added LED253: KT-0603R, footprint:LED0603-RD, F.Cu at (393.0, -90.3)
- added LED254: KT-0603R, footprint:LED0603-RD, F.Cu at (393.0, -87.7)
- added LED255: KT-0603R, footprint:LED0603-RD, F.Cu at (393.0, -85.0)
- added LED256: KT-0603R, footprint:LED0603-RD, F.Cu at (421.5, -90.3)
- added LED257: KT-0603R, footprint:LED0603-RD, F.Cu at (421.5, -87.7)
- added LED258: KT-0603R, footprint:LED0603-RD, F.Cu at (421.5, -85.0)
- added LED259: KT-0603R, footprint:LED0603-RD, F.Cu at (407.3, -90.3)
- added LED260: KT-0603R, footprint:LED0603-RD, F.Cu at (407.3, -87.7)
- added LED261: KT-0603R, footprint:LED0603-RD, F.Cu at (407.3, -85.0)
- added LED262: KT-0603R, footprint:LED0603-RD, F.Cu at (407.3, -69.5)
- added LED263: KT-0603R, footprint:LED0603-RD, F.Cu at (407.3, -66.9)
- added LED264: KT-0603R, footprint:LED0603-RD, F.Cu at (407.3, -64.2)
- added LED265: KT-0603R, footprint:LED0603-RD, F.Cu at (421.5, -69.5)
- added LED266: KT-0603R, footprint:LED0603-RD, F.Cu at (421.5, -66.9)
- added LED267: KT-0603R, footprint:LED0603-RD, F.Cu at (421.5, -64.2)
- added LED268: KT-0603R, footprint:LED0603-RD, F.Cu at (407.3, -59.1)
- added LED269: KT-0603R, footprint:LED0603-RD, F.Cu at (407.3, -56.5)
- added LED270: KT-0603R, footprint:LED0603-RD, F.Cu at (407.3, -53.8)
- added LED271: KT-0603R, footprint:LED0603-RD, F.Cu at (435.7, -69.5)
- added LED272: KT-0603R, footprint:LED0603-RD, F.Cu at (435.7, -66.9)
- added LED273: KT-0603R, footprint:LED0603-RD, F.Cu at (435.7, -64.2)
- added LED274: KT-0603R, footprint:LED0603-RD, F.Cu at (393.0, -100.7)
- added LED275: KT-0603R, footprint:LED0603-RD, F.Cu at (393.0, -98.1)
- added LED276: KT-0603R, footprint:LED0603-RD, F.Cu at (393.0, -95.4)
- added LED277: KT-0603R, footprint:LED0603-RD, F.Cu at (407.3, -100.7)
- added LED278: KT-0603R, footprint:LED0603-RD, F.Cu at (407.3, -98.1)
- added LED279: KT-0603R, footprint:LED0603-RD, F.Cu at (407.3, -95.4)
- added LED280: KT-0603R, footprint:LED0603-RD, F.Cu at (435.7, -100.7)
- added LED281: KT-0603R, footprint:LED0603-RD, F.Cu at (435.7, -98.1)
- added LED282: KT-0603R, footprint:LED0603-RD, F.Cu at (435.7, -95.4)
- added LED283: KT-0603R, footprint:LED0603-RD, F.Cu at (421.5, -100.7)
- added LED284: KT-0603R, footprint:LED0603-RD, F.Cu at (421.5, -98.1)
- added LED285: KT-0603R, footprint:LED0603-RD, F.Cu at (421.5, -95.4)
- added LED286: KT-0603R, footprint:LED0603-RD, F.Cu at (393.0, -69.5)
- added LED287: KT-0603R, footprint:LED0603-RD, F.Cu at (393.0, -66.9)
- added LED288: KT-0603R, footprint:LED0603-RD, F.Cu at (393.0, -64.2)
- added LED289: KT-0603R, footprint:LED0603-RD, F.Cu at (393.0, -59.1)
- added LED290: KT-0603R, footprint:LED0603-RD, F.Cu at (393.0, -56.5)
- added LED291: KT-0603R, footprint:LED0603-RD, F.Cu at (393.0, -53.8)
- added LED292: KT-0603R, footprint:LED0603-RD, F.Cu at (393.0, -38.3)
- added LED293: KT-0603R, footprint:LED0603-RD, F.Cu at (393.0, -35.7)
- added LED294: KT-0603R, footprint:LED0603-RD, F.Cu at (393.0, -33.0)
- added LED295: KT-0603R, footprint:LED0603-RD, F.Cu at (393.0, -48.7)
- added LED296: KT-0603R, footprint:LED0603-RD, F.Cu at (393.0, -46.1)
- added LED297: KT-0603R, footprint:LED0603-RD, F.Cu at (393.0, -43.4)
- added R156: 0603WAF2000T5E, footprint:R0603, F.Cu at (305.1, -26.1)
- added R157: 0603WAF2000T5E, footprint:R0603, F.Cu at (305.1, -23.7)
- added R158: 0805W8F2000T5E, footprint:R0805, F.Cu at (19.3, 130.6)
- added R159: 0805W8F0000T5E, footprint:R0805, F.Cu at (19.3, 133.6)
- added R160: 0603WAF2000T5E, footprint:R0603, F.Cu at (28.2, 135.7)
- added R161: 0805W8F0000T5E, footprint:R0805, F.Cu at (19.3, 136.6)
- added R162: 0603WAF2000T5E, footprint:R0603, F.Cu at (28.2, 138.1)
- added R163: 0603WAF2000T5E, footprint:R0603, F.Cu at (305.1, -39.0)
- added R164: 0603WAF2000T5E, footprint:R0603, F.Cu at (305.1, -36.5)
- added R165: 0603WAF2000T5E, footprint:R0603, F.Cu at (305.1, -34.1)
- added R166: 0603WAF2000T5E, footprint:R0603, F.Cu at (276.6, -91.0)
- added R167: 0603WAF2000T5E, footprint:R0603, F.Cu at (276.6, -88.5)
- added R168: 0603WAF2000T5E, footprint:R0603, F.Cu at (276.6, -86.1)
- added R169: 0603WAF2000T5E, footprint:R0603, F.Cu at (290.9, -91.0)
- added R170: 0603WAF2000T5E, footprint:R0603, F.Cu at (290.9, -88.5)
- added R171: 0603WAF2000T5E, footprint:R0603, F.Cu at (290.9, -86.1)
- added R172: 0603WAF2000T5E, footprint:R0603, F.Cu at (319.3, -91.0)
- added R173: 0603WAF2000T5E, footprint:R0603, F.Cu at (319.3, -88.5)
- added R174: 0603WAF2000T5E, footprint:R0603, F.Cu at (319.3, -86.1)
- added R175: 0603WAF2000T5E, footprint:R0603, F.Cu at (305.1, -91.0)
- added R176: 0603WAF2000T5E, footprint:R0603, F.Cu at (305.1, -88.5)
- added R177: 0603WAF2000T5E, footprint:R0603, F.Cu at (305.1, -86.1)
- added R178: 0603WAF2000T5E, footprint:R0603, F.Cu at (290.9, -70.2)
- added R179: 0603WAF2000T5E, footprint:R0603, F.Cu at (290.9, -67.7)
- added R180: 0603WAF2000T5E, footprint:R0603, F.Cu at (290.9, -65.3)
- added R181: 0603WAF2000T5E, footprint:R0603, F.Cu at (276.6, -39.0)
- added R182: 0603WAF2000T5E, footprint:R0603, F.Cu at (276.6, -36.5)
- added R183: 0603WAF2000T5E, footprint:R0603, F.Cu at (276.6, -34.1)
- added R184: 0603WAF2000T5E, footprint:R0603, F.Cu at (276.6, -28.6)
- added R185: 0603WAF2000T5E, footprint:R0603, F.Cu at (276.6, -26.1)
- added R186: 0603WAF2000T5E, footprint:R0603, F.Cu at (276.6, -23.7)
- added R187: 0603WAF2000T5E, footprint:R0603, F.Cu at (305.1, -59.8)
- added R188: 0603WAF2000T5E, footprint:R0603, F.Cu at (305.1, -57.3)
- added R189: 0603WAF2000T5E, footprint:R0603, F.Cu at (305.1, -54.9)
- added R190: 0603WAF2000T5E, footprint:R0603, F.Cu at (290.9, -59.8)
- added R191: 0603WAF2000T5E, footprint:R0603, F.Cu at (290.9, -57.3)
- added R192: 0603WAF2000T5E, footprint:R0603, F.Cu at (290.9, -54.9)
- added R193: 0603WAF2000T5E, footprint:R0603, F.Cu at (319.3, -28.6)
- added R194: 0603WAF2000T5E, footprint:R0603, F.Cu at (319.3, -26.1)
- added R195: 0603WAF2000T5E, footprint:R0603, F.Cu at (319.3, -23.7)
- added R196: 0603WAF2000T5E, footprint:R0603, F.Cu at (276.6, -101.4)
- added R197: 0603WAF2000T5E, footprint:R0603, F.Cu at (276.6, -98.9)
- added R198: 0603WAF2000T5E, footprint:R0603, F.Cu at (276.6, -96.5)
- added R199: 0603WAF2000T5E, footprint:R0603, F.Cu at (290.9, -101.4)
- added R200: 0603WAF2000T5E, footprint:R0603, F.Cu at (290.9, -98.9)
- added R201: 0603WAF2000T5E, footprint:R0603, F.Cu at (290.9, -96.5)
- added R202: 0603WAF2000T5E, footprint:R0603, F.Cu at (319.3, -101.4)
- added R203: 0603WAF2000T5E, footprint:R0603, F.Cu at (319.3, -98.9)
- added R204: 0603WAF2000T5E, footprint:R0603, F.Cu at (319.3, -96.5)
- added R205: 0603WAF2000T5E, footprint:R0603, F.Cu at (305.1, -101.4)
- added R206: 0603WAF2000T5E, footprint:R0603, F.Cu at (305.1, -98.9)
- added R207: 0603WAF2000T5E, footprint:R0603, F.Cu at (305.1, -96.5)
- added R208: 0603WAF2000T5E, footprint:R0603, F.Cu at (319.3, -70.2)
- added R209: 0603WAF2000T5E, footprint:R0603, F.Cu at (319.3, -67.7)
- added R210: 0603WAF2000T5E, footprint:R0603, F.Cu at (319.3, -65.3)
- added R211: 0603WAF2000T5E, footprint:R0603, F.Cu at (276.6, -49.4)
- added R212: 0603WAF2000T5E, footprint:R0603, F.Cu at (276.6, -46.9)
- added R213: 0603WAF2000T5E, footprint:R0603, F.Cu at (276.6, -44.5)
- added R214: 0603WAF2000T5E, footprint:R0603, F.Cu at (319.3, -59.8)
- added R215: 0603WAF2000T5E, footprint:R0603, F.Cu at (319.3, -57.3)
- added R216: 0603WAF2000T5E, footprint:R0603, F.Cu at (319.3, -54.9)
- added R217: 0603WAF2000T5E, footprint:R0603, F.Cu at (319.3, -39.0)
- added R218: 0603WAF2000T5E, footprint:R0603, F.Cu at (319.3, -36.5)
- added R219: 0603WAF2000T5E, footprint:R0603, F.Cu at (319.3, -34.1)
- added R220: 0603WAF2000T5E, footprint:R0603, F.Cu at (276.6, -59.8)
- added R221: 0603WAF2000T5E, footprint:R0603, F.Cu at (276.6, -57.3)
- added R222: 0603WAF2000T5E, footprint:R0603, F.Cu at (276.6, -54.9)
- added R223: 0603WAF2000T5E, footprint:R0603, F.Cu at (319.3, -49.4)
- added R224: 0603WAF2000T5E, footprint:R0603, F.Cu at (319.3, -46.9)
- added R225: 0603WAF2000T5E, footprint:R0603, F.Cu at (319.3, -44.5)
- added R226: 0603WAF2000T5E, footprint:R0603, F.Cu at (305.1, -70.2)
- added R227: 0603WAF2000T5E, footprint:R0603, F.Cu at (305.1, -67.7)
- added R228: 0603WAF2000T5E, footprint:R0603, F.Cu at (305.1, -65.3)
- added R229: 0603WAF2000T5E, footprint:R0603, F.Cu at (276.6, -80.6)
- added R230: 0603WAF2000T5E, footprint:R0603, F.Cu at (276.6, -78.1)
- added R231: 0603WAF2000T5E, footprint:R0603, F.Cu at (276.6, -75.7)
- added R232: 0603WAF2000T5E, footprint:R0603, F.Cu at (290.9, -80.6)
- added R233: 0603WAF2000T5E, footprint:R0603, F.Cu at (290.9, -78.1)
- added R234: 0603WAF2000T5E, footprint:R0603, F.Cu at (290.9, -75.7)
- added R235: 0603WAF2000T5E, footprint:R0603, F.Cu at (319.3, -80.6)
- added R236: 0603WAF2000T5E, footprint:R0603, F.Cu at (319.3, -78.1)
- added R237: 0603WAF2000T5E, footprint:R0603, F.Cu at (319.3, -75.7)
- added R238: 0603WAF2000T5E, footprint:R0603, F.Cu at (305.1, -80.6)
- added R239: 0603WAF2000T5E, footprint:R0603, F.Cu at (305.1, -78.1)
- added R240: 0603WAF2000T5E, footprint:R0603, F.Cu at (305.1, -75.7)
- added R241: 0603WAF2000T5E, footprint:R0603, F.Cu at (290.9, -49.4)
- added R242: 0603WAF2000T5E, footprint:R0603, F.Cu at (290.9, -46.9)
- added R243: 0603WAF2000T5E, footprint:R0603, F.Cu at (290.9, -44.5)
- added R244: 0603WAF2000T5E, footprint:R0603, F.Cu at (290.9, -39.0)
- added R245: 0603WAF2000T5E, footprint:R0603, F.Cu at (290.9, -36.5)
- added R246: 0603WAF2000T5E, footprint:R0603, F.Cu at (290.9, -34.1)
- added R247: 0603WAF2000T5E, footprint:R0603, F.Cu at (305.1, -49.4)
- added R248: 0603WAF2000T5E, footprint:R0603, F.Cu at (305.1, -46.9)
- added R249: 0603WAF2000T5E, footprint:R0603, F.Cu at (305.1, -44.5)
- added R250: 0603WAF2000T5E, footprint:R0603, F.Cu at (290.9, -28.6)
- added R251: 0603WAF2000T5E, footprint:R0603, F.Cu at (290.9, -26.1)
- added R252: 0603WAF2000T5E, footprint:R0603, F.Cu at (290.9, -23.7)
- added R253: 0603WAF2000T5E, footprint:R0603, F.Cu at (276.6, -70.2)
- added R254: 0603WAF2000T5E, footprint:R0603, F.Cu at (276.6, -67.7)
- added R255: 0603WAF2000T5E, footprint:R0603, F.Cu at (276.6, -65.3)
- added R256: 0603WAF2000T5E, footprint:R0603, F.Cu at (382.7, -80.0)
- added R257: 0603WAF2000T5E, footprint:R0603, F.Cu at (382.7, -77.6)
- added R258: 0603WAF2000T5E, footprint:R0603, F.Cu at (382.7, -75.1)
- added R259: 0603WAF2000T5E, footprint:R0603, F.Cu at (382.7, -69.6)
- added R260: 0603WAF2000T5E, footprint:R0603, F.Cu at (382.7, -67.2)
- added R261: 0603WAF2000T5E, footprint:R0603, F.Cu at (382.7, -64.7)
- added R262: 0603WAF2000T5E, footprint:R0603, F.Cu at (382.7, -48.8)
- added R263: 0603WAF2000T5E, footprint:R0603, F.Cu at (382.7, -46.4)
- added R264: 0603WAF2000T5E, footprint:R0603, F.Cu at (382.7, -43.9)
- added R265: 0603WAF2000T5E, footprint:R0603, F.Cu at (382.7, -59.2)
- added R266: 0603WAF2000T5E, footprint:R0603, F.Cu at (382.7, -56.8)
- added R267: 0603WAF2000T5E, footprint:R0603, F.Cu at (382.7, -54.3)
- added R268: 0603WAF2000T5E, footprint:R0603, F.Cu at (397.0, -28.0)
- added R269: 0603WAF2000T5E, footprint:R0603, F.Cu at (397.0, -25.6)
- added R270: 0603WAF2000T5E, footprint:R0603, F.Cu at (397.0, -23.1)
- added R271: 0603WAF2000T5E, footprint:R0603, F.Cu at (411.2, -80.0)
- added R272: 0603WAF2000T5E, footprint:R0603, F.Cu at (411.2, -77.6)
- added R273: 0603WAF2000T5E, footprint:R0603, F.Cu at (411.2, -75.1)
- added R274: 0603WAF2000T5E, footprint:R0603, F.Cu at (439.6, -80.0)
- added R275: 0603WAF2000T5E, footprint:R0603, F.Cu at (439.6, -77.6)
- added R276: 0603WAF2000T5E, footprint:R0603, F.Cu at (439.6, -75.1)
- added R277: 0603WAF2000T5E, footprint:R0603, F.Cu at (425.4, -80.0)
- added R278: 0603WAF2000T5E, footprint:R0603, F.Cu at (425.4, -77.6)
- added R279: 0603WAF2000T5E, footprint:R0603, F.Cu at (425.4, -75.1)
- added R280: 0603WAF2000T5E, footprint:R0603, F.Cu at (397.0, -80.0)
- added R281: 0603WAF2000T5E, footprint:R0603, F.Cu at (397.0, -77.6)
- added R282: 0603WAF2000T5E, footprint:R0603, F.Cu at (397.0, -75.1)
- added R283: 0603WAF2000T5E, footprint:R0603, F.Cu at (382.7, -90.4)
- added R284: 0603WAF2000T5E, footprint:R0603, F.Cu at (382.7, -88.0)
- added R285: 0603WAF2000T5E, footprint:R0603, F.Cu at (382.7, -85.5)
- added R286: 0603WAF2000T5E, footprint:R0603, F.Cu at (439.6, -90.4)
- added R287: 0603WAF2000T5E, footprint:R0603, F.Cu at (439.6, -88.0)
- added R288: 0603WAF2000T5E, footprint:R0603, F.Cu at (439.6, -85.5)
- added R289: 0603WAF2000T5E, footprint:R0603, F.Cu at (382.7, -38.4)
- added R290: 0603WAF2000T5E, footprint:R0603, F.Cu at (382.7, -36.0)
- added R291: 0603WAF2000T5E, footprint:R0603, F.Cu at (382.7, -33.5)
- added R292: 0603WAF2000T5E, footprint:R0603, F.Cu at (411.2, -48.8)
- added R293: 0603WAF2000T5E, footprint:R0603, F.Cu at (411.2, -46.4)
- added R294: 0603WAF2000T5E, footprint:R0603, F.Cu at (411.2, -43.9)
- added R295: 0603WAF2000T5E, footprint:R0603, F.Cu at (411.2, -38.4)
- added R296: 0603WAF2000T5E, footprint:R0603, F.Cu at (411.2, -36.0)
- added R297: 0603WAF2000T5E, footprint:R0603, F.Cu at (411.2, -33.5)
- added R298: 0603WAF2000T5E, footprint:R0603, F.Cu at (382.7, -100.8)
- added R299: 0603WAF2000T5E, footprint:R0603, F.Cu at (382.7, -98.4)
- added R300: 0603WAF2000T5E, footprint:R0603, F.Cu at (382.7, -95.9)
- added R301: 0603WAF2000T5E, footprint:R0603, F.Cu at (411.2, -28.0)
- added R302: 0603WAF2000T5E, footprint:R0603, F.Cu at (411.2, -25.6)
- added R303: 0603WAF2000T5E, footprint:R0603, F.Cu at (411.2, -23.1)
- added R304: 0603WAF2000T5E, footprint:R0603, F.Cu at (382.7, -28.0)
- added R305: 0603WAF2000T5E, footprint:R0603, F.Cu at (382.7, -25.6)
- added R306: 0603WAF2000T5E, footprint:R0603, F.Cu at (382.7, -23.1)
- added R307: 0603WAF2000T5E, footprint:R0603, F.Cu at (397.0, -90.4)
- added R308: 0603WAF2000T5E, footprint:R0603, F.Cu at (397.0, -88.0)
- added R309: 0603WAF2000T5E, footprint:R0603, F.Cu at (397.0, -85.5)
- added R310: 0603WAF2000T5E, footprint:R0603, F.Cu at (425.4, -90.4)
- added R311: 0603WAF2000T5E, footprint:R0603, F.Cu at (425.4, -88.0)
- added R312: 0603WAF2000T5E, footprint:R0603, F.Cu at (425.4, -85.5)
- added R313: 0603WAF2000T5E, footprint:R0603, F.Cu at (411.2, -90.4)
- added R314: 0603WAF2000T5E, footprint:R0603, F.Cu at (411.2, -88.0)
- added R315: 0603WAF2000T5E, footprint:R0603, F.Cu at (411.2, -85.5)
- added R316: 0603WAF2000T5E, footprint:R0603, F.Cu at (411.2, -69.6)
- added R317: 0603WAF2000T5E, footprint:R0603, F.Cu at (411.2, -67.2)
- added R318: 0603WAF2000T5E, footprint:R0603, F.Cu at (411.2, -64.7)
- added R319: 0603WAF2000T5E, footprint:R0603, F.Cu at (425.4, -69.6)
- added R320: 0603WAF2000T5E, footprint:R0603, F.Cu at (425.4, -67.2)
- added R321: 0603WAF2000T5E, footprint:R0603, F.Cu at (425.4, -64.7)
- added R322: 0603WAF2000T5E, footprint:R0603, F.Cu at (411.2, -59.2)
- added R323: 0603WAF2000T5E, footprint:R0603, F.Cu at (411.2, -56.8)
- added R324: 0603WAF2000T5E, footprint:R0603, F.Cu at (411.2, -54.3)
- added R325: 0603WAF2000T5E, footprint:R0603, F.Cu at (439.6, -69.6)
- added R326: 0603WAF2000T5E, footprint:R0603, F.Cu at (439.6, -67.2)
- added R327: 0603WAF2000T5E, footprint:R0603, F.Cu at (439.6, -64.7)
- added R328: 0603WAF2000T5E, footprint:R0603, F.Cu at (397.0, -100.8)
- added R329: 0603WAF2000T5E, footprint:R0603, F.Cu at (397.0, -98.4)
- added R330: 0603WAF2000T5E, footprint:R0603, F.Cu at (397.0, -95.9)
- added R331: 0603WAF2000T5E, footprint:R0603, F.Cu at (411.2, -100.8)
- added R332: 0603WAF2000T5E, footprint:R0603, F.Cu at (411.2, -98.4)
- added R333: 0603WAF2000T5E, footprint:R0603, F.Cu at (411.2, -95.9)
- added R334: 0603WAF2000T5E, footprint:R0603, F.Cu at (439.6, -100.8)
- added R335: 0603WAF2000T5E, footprint:R0603, F.Cu at (439.6, -98.4)
- added R336: 0603WAF2000T5E, footprint:R0603, F.Cu at (439.6, -95.9)
- added R337: 0603WAF2000T5E, footprint:R0603, F.Cu at (425.4, -100.8)
- added R338: 0603WAF2000T5E, footprint:R0603, F.Cu at (425.4, -98.4)
- added R339: 0603WAF2000T5E, footprint:R0603, F.Cu at (425.4, -95.9)
- added R340: 0603WAF2000T5E, footprint:R0603, F.Cu at (397.0, -69.6)
- added R341: 0603WAF2000T5E, footprint:R0603, F.Cu at (397.0, -67.2)
- added R342: 0603WAF2000T5E, footprint:R0603, F.Cu at (397.0, -64.7)
- added R343: 0603WAF2000T5E, footprint:R0603, F.Cu at (397.0, -59.2)
- added R344: 0603WAF2000T5E, footprint:R0603, F.Cu at (397.0, -56.8)
- added R345: 0603WAF2000T5E, footprint:R0603, F.Cu at (397.0, -54.3)
- added R346: 0603WAF2000T5E, footprint:R0603, F.Cu at (397.0, -38.4)
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- renumbered B102 to B101, B101 to B102, C127 to C102, C109 to C104, C111 to C105, C110 to C106, C112 to C107, C113 to C108, C115 to C109, C114 to C110, C128 to C111, C118 to C112, C116 to C113, C119 to C114, C117 to C115, H103 to H102, H102 to H103, J107 to J101, J111 to J102, J115 to J103, J109 to J105, J113 to J106, J102 to J107, J117 to J108, J119 to J109, J123 to J110, J125 to J111, J127 to J112, J128 to J113, J129 to J114, J101 to J115, J120 to J116, J103 to J117, J105 to J118, J108 to J119, J110 to J120, J112 to J121, J114 to J122, J116 to J123, J118 to J124, J121 to J125, J124 to J126, J126 to J127, J106 to J128, J122 to J129, J150 to J135, J151 to J136, J152 to J137, J153 to J138, J154 to J139, J135 to J140, J136 to J141, J137 to J142, J138 to J143, J139 to J144, J155 to J145, J156 to J146, J157 to J147, J158 to J148, J140 to J149, J141 to J150, J142 to J151, J143 to J152, J144 to J153, J145 to J154, J146 to J155, J147 to J156, J148 to J157, J149 to J158, LED103 to LED102, LED102 to LED103, P103 to P102, P105 to P103, P102 to P104, P104 to P105, R105 to R101, R109 to R102, R111 to R103, R108 to R104, R110 to R105, R104 to R106, R157 to R107, R156 to R108, R158 to R109, R152 to R110, R150 to R111, R101 to R112, R159 to R113, R151 to R114, R106 to R115, R112 to R116, R107 to R117, R102 to R118, R103 to R119, R115 to R120, R119 to R121, R117 to R122, R114 to R123, R118 to R124, R116 to R125, R141 to R126, R142 to R127, R143 to R128, R144 to R129, R145 to R130, R121 to R131, R122 to R132, R123 to R133, R124 to R134, R125 to R135, R146 to R136, R147 to R137, R148 to R138, R149 to R139, R126 to R140, R127 to R141, R128 to R142, R129 to R143, R130 to R144, R131 to R145, R132 to R146, R133 to R147, R134 to R148, R135 to R149, R136 to R150, R137 to R151, R138 to R152, R139 to R153, R140 to R154, U104 to U101, U105 to U102, U101 to U103, U103 to U104, U180 to U105, U102 to U106, U136 to U108, U138 to U109, U137 to U110, U139 to U111, U140 to U112, U142 to U113, U141 to U114, U143 to U115, U144 to U116, U147 to U117, U145 to U118, U148 to U119, U146 to U120, c108 to c101
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Connections:
- BUZ101 pad 1: /Bottom/VDD -> Net-(LED107-A)
- BUZ101 pad 2: Net-(U106-D) -> Net-(U124-D)
- C103 pad 1: GND -> /Bottom/+3.3V
- C103 pad 2: /Bottom/VDD -> GND
- C120 pad 1: /Top/GND -> /Top/+3.3V_LEDS
- C120 pad 2: /Top/VDD -> /Top/GND
- C121 pad 1: /Top/GND -> /Bottom/+3.3V
- C121 pad 2: /Top/VDD -> GND
- C122 pad 1: /Top/GND -> /Top/+3.3V_LEDS
- C122 pad 2: /Top/VDD -> /Top/GND
- C123 pad 1: /Top/GND -> /Top/+3.3V_LEDS
- C123 pad 2: /Top/VDD -> /Top/GND
- C124 pad 1: /Top/GND -> /Bottom/+3.3V
- C124 pad 2: /Top/VDD -> GND
- C125 pad 1: /Top/GND -> /Top/+3.3V_LEDS
- C125 pad 2: /Top/VDD -> /Top/GND
- C126 pad 1: /Top/GND -> /Bottom/+3.3V
- C126 pad 2: /Top/VDD -> GND
- C129 pad 1: /Bottom/VDD -> /Top/+3.3V_LEDS
- C129 pad 2: GND -> /Top/GND
- P101 pad 1: /Top/VDD -> /Top/+3.3V_LEDS
- P101 pad 3: /Top/VDD -> /SOFTSPI_CLK_LID
- P101 pad 5: /Top/VDD -> /SOFTSPI_RST_LID
- P101 pad 7: /Top/VDD -> /SOFTSPI_CSn_LID
- P101 pad 9: /Top/LED_DATA_IN -> /SER_DATA_IN_0
- P102 pad 7: unconnected-(P103-Pad7) -> /Top/VDD
- P102 pad 9: unconnected-(P103-Pad9) -> /Top/VDD
- P104 pad 1: /Bottom/VDD -> /Bottom/+3.3V
- P104 pad 3: /Bottom/VDD -> /SOFTSPI_CLK_BOT
- P104 pad 5: /Bottom/VDD -> /SOFTSPI_RST_BOT
- P104 pad 7: /Bottom/VDD -> /SOFTSPI_CSn_BOT
- P104 pad 9: /Bottom/LED_DATA_OUT -> /SER_DATA_OUT_8_BOT
- P105 pad 7: unconnected-(P104-Pad7) -> /Bottom/VDD
- P105 pad 9: unconnected-(P104-Pad9) -> /Bottom/VDD
- R155 pad 1: Net-(U106-D) -> Net-(LED104-A)
- R155 pad 2: /Bottom/VDD -> /Bottom/LEDs_Bottom/VDD
- U104 pad 16: /Bottom/+3.3V -> unconnected-(U104-GPIO12-Pad16)
- U104 pad 20: /Bottom/LED_DATA_IN -> /SOFTSPI_CSn_BOT
- U104 pad 31: unconnected-(U103-GPIO26_ADC0-Pad31) -> /SOFTSPI_CLK_BOT
- U104 pad 32: unconnected-(U103-GPIO27_ADC1-Pad32) -> /Bottom/SOFTSPI_MOSI
- U104 pad 34: unconnected-(U103-GPIO28_ADC2-Pad34) -> /Bottom/SOFTSPI_MISO
- U107 pad 1: /Bottom/LEDs Sheet/LED_DATA_IN -> /Bottom/LEDs_Bottom/LEDS_discreet/LED_single/LED_GREEN
- U107 pad 2: /Bottom/VDD -> /Bottom/LEDs_Bottom/LEDS_discreet/LED_single1/LED_RED
- U107 pad 3: Net-(U107-DO) -> /Bottom/LEDs_Bottom/LEDS_discreet/LED_single1/LED_GREEN
- U107 pad 4: GND -> /Bottom/LEDs_Bottom/LEDS_discreet/LED_single2/LED_RED
- U121 pad 1: Net-(U120-DO) -> /Bottom/LEDs_Bottom/LEDS_discreet/LED_single1/LED_RED
- U121 pad 2: /Bottom/VDD -> GND
- U121 pad 3: Net-(U121-DO) -> Net-(LED104-K)
- U122 pad 1: Net-(U121-DO) -> /Bottom/LEDs_Bottom/LEDS_discreet/LED_single1/LED_GREEN
- U122 pad 2: /Bottom/VDD -> GND
- U122 pad 3: Net-(U122-DO) -> Net-(LED106-K)
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Routing:
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- removed copper zone on B.Cu, net /Top/GND
- removed copper zone on F.Cu, net /Top/GND
- removed copper zone on B.Cu, net GND
- removed copper zone on F.Cu, net GND
Other:
- board text added: "Kabooom Box"
- board text removed: "Alfreds Kabooom Box"
