File: KiCad/Kaboom_box.kicad_pcb (KiCad board)
At the start: 2 copper layers, 333.9 x 141.1 mm, 723 parts, among them J101 2mm_clamp, J102 2mm_clamp, J103 2mm_clamp, J104 2mm_clamp, J105 2mm_clamp, J106 2mm_clamp, J107 2mm_clamp, J108 2mm_clamp, J109 2mm_clamp, J110 2mm_clamp, J111 2mm_clamp, J112 2mm_clamp, J113 2mm_clamp, J114 2mm_clamp, J115 2mm_clamp, J116 2mm_clamp, J117 2mm_clamp, J118 2mm_clamp, J119 2mm_clamp, J120 2mm_clamp, J121 2mm_clamp, J122 2mm_clamp, J123 2mm_clamp, J124 2mm_clamp, J125 2mm_clamp, J126 2mm_clamp, J127 2mm_clamp, J128 2mm_clamp, J129 2mm_clamp, J130 2mm_clamp, J131 2mm_clamp, J132 2mm_clamp, J133 2mm_clamp, J134 2mm_clamp, J135 2mm_clamp, J136 2mm_clamp, J137 2mm_clamp, J138 2mm_clamp, J139 2mm_clamp, J140 2mm_clamp, J141 2mm_clamp, J142 2mm_clamp, J143 2mm_clamp, J144 2mm_clamp, J145 2mm_clamp, J146 2mm_clamp, J147 2mm_clamp, J148 2mm_clamp, J149 2mm_clamp, J150 2mm_clamp, J151 2mm_clamp, J152 2mm_clamp, J153 2mm_clamp, J154 2mm_clamp, J155 2mm_clamp, J156 2mm_clamp, J157 2mm_clamp, J158 2mm_clamp, J159 Screw_Terminal_01x02, P101 HDR-IDC-2_54-2X5P, P102 HDR-IDC-2_54-2X5P, P103 HDR-IDC-2_54-2X5P, P104 HDR-IDC-2_54-2X5P, P105 HDR-IDC-2_54-2X5P, P106 HDR-IDC-2_54-2X5P, U101 TS-1187A-B-A-B, U102 TS-1187A-B-A-B, U103 SS54_C22452, U104 RaspberryPi_Pico, U105 AO3400A, U106 EC12E1220813, U107 74HC595D,118, U108 74HC595D,118, U109 74HC595D,118, U110 74HC595D,118, U111 74HC595D,118, U112 MT-0-103-F001-T000-RS+PJ, U113 MT-0-103-F001-T000-RS+PJ, U114 MT-0-103-F001-T000-RS+PJ, U115 PZ254V-11-04P_C2691448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

Commit message: WIP
Parts:
- J159: moved to B.Cu
- moved U207 703.8 mm to (869.5, -537.1), turned to 150 degrees
- moved U206 697.3 mm to (867.8, -533.9), turned to 150 degrees
- moved LED216 696.3 mm to (875.9, -524.3), turned to -120 degrees
- moved LED214 695.0 mm to (871.4, -532.2)
- moved R268 693.5 mm to (876.0, -529.5), turned to -60 degrees
- moved R269 689.1 mm to (866.9, -529.5), turned to 60 degrees
- moved R270 688.3 mm to (871.4, -521.7), turned to 180 degrees
- moved LED215 688.1 mm to (866.9, -524.3), turned to 120 degrees
- moved U229 638.9 mm to (863.9, -465.4), turned to 150 degrees
- moved U228 632.6 mm to (862.1, -462.3), turned to 150 degrees
- moved LED249 631.9 mm to (870.3, -452.7), turned to -120 degrees
- moved LED247 630.4 mm to (865.7, -460.6)
- moved R301 629.0 mm to (870.3, -457.9), turned to -60 degrees
- moved U265 625.5 mm to (767.1, -541.9), turned to 150 degrees
- moved R302 624.1 mm to (861.2, -457.9), turned to 60 degrees
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Connections:
- U104 pad 16: unconnected-(U104-GPIO12-Pad16) -> /SOFTSPI_RST_BOT
Routing:
- net /Bottom/LEDs_Bottom/VDD: track 0.00 -> 154.2 mm, vias 0 -> 128
- net /Top/VDD: track 126.8 -> 281.0 mm, vias 0 -> 128
- net Net-(J128-Pin_1): track 117.4 -> 0.00 mm
- net Net-(J115-Pin_1): track 117.4 -> 0.00 mm
- net Net-(J129-Pin_1): track 117.4 -> 0.00 mm
- net Net-(J116-Pin_1): track 117.4 -> 0.00 mm
- net Net-(J117-Pin_1): track 96.8 -> 0.00 mm
- net Net-(J124-Pin_1): track 96.8 -> 0.00 mm
- net Net-(J108-Pin_1): track 96.8 -> 0.00 mm
- net Net-(J104-Pin_1): track 96.8 -> 0.00 mm
- net /Bottom/VDD: track 154.2 -> 58.6 mm
- net Net-(J118-Pin_1): track 82.8 -> 0.00 mm
- net Net-(J125-Pin_1): track 82.7 -> 0.00 mm
- net Net-(J109-Pin_1): track 82.7 -> 0.00 mm
- net Net-(J101-Pin_1): track 82.7 -> 0.00 mm
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- removed copper zone on F.Cu, net Net-(R107-Pad1)
Other:
- board size 333.9 x 141.1 mm -> 314.7 x 142.9 mm
