File: KiCad/Bottom.kicad_sch (KiCad schematic)
At the start: 32 parts, among them U101 TS-1187A-B-A-B, U102 TS-1187A-B-A-B, U103 SS54_C22452, U104 RaspberryPi_Pico, U105 AO3400A, U106 EC12E1220813

Commit message: WIP
Connections:
- net SOFTSPI_RST: now also U104.16 (GPIO12)
